File: hw/fanctl2.sch (KiCad schematic (older format))
At the start: 3 parts, among them U0 ULN2003

Commit message: PCB pretty much done.
I changed the size so it would be smaller than 10x10 cm, otherwise it's
absurdly expensive to have it made.
Parts:
- added C0, C1, C10, C11, C12, C13, C14, C2, C3, C4, C5, C6, C7, C8, C9: Decoupler, Capacitors_ThroughHole:C_Disc_D3_P2.5, symbol Decoupler
- added D0, D1: ZENER, Diodes_ThroughHole:Diode_DO-35_SOD27_Horizontal_RM10, symbol ZENER
- added D2, D3, D4, D5, D6: LED, LEDs:LED-5MM, symbol LED
- added F1: F_Small, Resistors_ThroughHole:Resistor_Horizontal_RM10mm, symbol F_Small
- added FAN0, FAN1, FAN2, FAN3, FAN4, FAN5: 4PIN_FAN, ab2_header:AB2_HDR_M04-1V_CPU_FAN, symbol 4PIN_FAN
- added I2C0: I2C_HDR, Pin_Headers:Pin_Header_Straight_2x02, symbol I2C_HDR
- added ICSP0: Prog_con, Pin_Headers:Pin_Header_Straight_2x03, symbol Prog_con
- added JP0, JP1, JP2, JP3, JP4, JP5: Jumper_NC_Small, Pin_Headers:Pin_Header_Straight_1x02, symbol Jumper_NC_Small
- added JP6: Jumper_NO_Small, Pin_Headers:Pin_Header_Straight_1x02, symbol Jumper_NO_Small
- added L1: INDUCTOR_SMALL, Inductors:INDUCTOR_V, symbol INDUCTOR_SMALL
- added P0: CONN_01X02, Pin_Headers:Pin_Header_Straight_1x02, symbol CONN_01X02
- added P1: MOLEX_PWR, ab2_power:AB2_ATX_PSU-4PIN-V, symbol MOLEX_PWR
- added Q0, Q1, Q2, Q3, Q4, Q5: FAN_PMOS, TO_SOT_Packages_THT:TO-220_Neutral123_Vertical, symbol FAN_PMOS
- added Q6: BC413, TO_SOT_Packages_THT:TO-92_Inline_Narrow_Oval, symbol BC413
- added R0, R1, R10, R11, R12, R13, R14, R15, R19, R2, R3, R4, R5, R6, R7, R8, R9: FANCTL2_R, Resistors_ThroughHole:Resistor_Horizontal_RM10mm, symbol FANCTL2_R
- added TEMP0: TMP_SNSR_HDR, Pin_Headers:Pin_Header_Straight_2x10, symbol TMP_SNSR_HDR
- added U1: 7400, Housings_DIP:DIP-14_W7.62mm, symbol 7400
- added USB0: USB_HDR, Pin_Headers:Pin_Header_Angled_1x04, symbol USB_HDR
- added Y0: Crystal_Small, Crystals:Crystal_HC49-U_Vertical, symbol Crystal_Small
- MCU0: footprint DIL28 -> Housings_DIP:DIP-28_W7.62mm
- MPLX0: footprint Housings_DIP:DIP-24_W10.16mm -> Housings_DIP:DIP-24_W7.62mm; Manu1 (none) -> Texas Instruments; Manu1 part no (none) -> CD47HC4067E; Manufacturer Texas Instruments -> (none); Part No CD47HC4067E -> (none); Supp1 (none) -> Farnell; Supp1 part no (none) -> 1740160
- U0: footprint (none) -> Housings_DIP:DIP-16_W7.62mm; Manu1 (none) -> TI; Supp1 (none) -> Farnell; Supp1 part no (none) -> 1470512
Connections:
- net labels added: +12V, +5V, GND, LED0, LED1, LED2, PWM0, PWM1, PWM12_0, PWM12_1, PWM12_2, PWM12_3, PWM12_4, PWM12_5, PWM2, PWM3, PWM4, PWM5, SEL0, SEL1, SEL2, SEL3, SENS0, TACH0, TACH1, TACH2, TACH3, TACH4, TACH5
- wire segments 0 -> 174
- no-connect marks 0 -> 6
Other:
- moved on the sheet: MCU0, U0

Commit message: Add a resistor.
Parts:
- removed U0: ULN2003, Housings_DIP:DIP-16_W7.62mm, symbol ULN2003
- added R16: R, Resistors_ThroughHole:Resistor_Horizontal_RM10mm, symbol R
- added U0: F2_ULN2003, Housings_DIP:DIP-16_W7.62mm, symbol F2_ULN2003
Connections:
- wire segments 174 -> 175
Changed lines of the file:
@@
 $EndDescr
-$Comp
-L ULN2003 U0
-U 1 1 56845E25
-P 2900 4950
-F 0 "U0" H 2900 5050 50  0000 C CNN
-F 1 "ULN2003" H 2900 4850 50  0000 C CNN
-F 2 "Housings_DIP:DIP-16_W7.62mm" H 2900 4950 50  0001 C CNN
-F 3 "" H 2900 4950 50  0000 C CNN
-F 4 "TI" H 2900 4950 60  0001 C CNN "Manu1"
-F 5 "Farnell" H 2900 4950 60  0001 C CNN "Supp1"
-F 6 "1470512" H 2900 4950 60  0001 C CNN "Supp1 part no"
-	1    2900 4950
-	0    1    1    0
-$EndComp
 $Comp
 L Multiplexer_16:1 MPLX0
@@
 	9850 1250 9850 1300
 NoConn ~ 6050 2650
+$Comp
+L F2_ULN2003 U0
+U 1 1 56898C90
+P 2900 4950
+F 0 "U0" H 2900 5050 50  0000 C CNN
+F 1 "F2_ULN2003" V 2900 4700 50  0000 C CNN
+F 2 "Housings_DIP:DIP-16_W7.62mm" H 2900 4950 50  0001 C CNN
+F 3 "" H 2900 4950 50  0000 C CNN
+	1    2900 4950
+	0    1    1    0
+$EndComp
+$Comp
+L R R16
+U 1 1 56898F5F
+P 2200 4450
+F 0 "R16" V 2280 4450 50  0000 C CNN
+F 1 "R" V 2200 4450 50  0000 C CNN
+F 2 "Resistors_ThroughHole:Resistor_Horizontal_RM10mm" V 2130 4450 50  0001 C CNN
+F 3 "" H 2200 4450 50  0000 C CNN
+F 4 "1.5k" V 2200 4450 60  0001 C CNN "R"
+	1    2200 4450
+	1    0    0    -1
+$EndComp
+Wire Wire Line
+	2500 4300 2200 4300
+$Comp
+L GND #PWR049
+U 1 1 5689913C
+P 2200 4600
+F 0 "#PWR049" H 2200 4350 50  0001 C CNN
+F 1 "GND" H 2200 4450 50  0000 C CNN
+F 2 "" H 2200 4600 50  0000 C CNN
+F 3 "" H 2200 4600 50  0000 C CNN
+	1    2200 4600
+	1    0    0    -1
+$EndComp
 $EndSCHEMATC

Commit message: Lots of changes
Parts:
- removed C10, C12: Decoupler, Capacitors_ThroughHole:C_Disc_D3_P2.5, symbol Decoupler
- removed JP0, JP1, JP2, JP3, JP4, JP5: Jumper_NC_Small, Pin_Headers:Pin_Header_Straight_1x02, symbol Jumper_NC_Small
- removed Q0, Q1, Q2, Q3, Q4, Q5: FAN_PMOS, TO_SOT_Packages_THT:TO-220_Neutral123_Vertical, symbol FAN_PMOS
- removed R15, R19: FANCTL2_R, Resistors_ThroughHole:Resistor_Horizontal_RM10mm, symbol FANCTL2_R
- removed R16: R, Resistors_ThroughHole:Resistor_Horizontal_RM10mm, symbol R
- removed U0: F2_ULN2003, Housings_DIP:DIP-16_W7.62mm, symbol F2_ULN2003
- added D?: D, symbol D
- added Q0, Q1, Q2, Q3, Q4, Q5: FAN_NMOS, symbol FAN_NMOS
- added R? (x2): R, symbol R
- added RR?: RR9, symbol RR9
Connections:
- net labels removed: PWM12_0, PWM12_1, PWM12_2, PWM12_3, PWM12_4, PWM12_5
- wire segments 175 -> 177
- no-connect marks 6 -> 4
Other:
- moved on the sheet: C0, C1, C14, C2, C3, C4, C5, FAN0, FAN1, FAN2, FAN3, FAN4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

Commit message: Tons of changes
Parts:
- removed P0: CONN_01X02, Pin_Headers:Pin_Header_Straight_1x02, symbol CONN_01X02
- removed Q0: FAN_NMOS, symbol FAN_NMOS
- removed R0, R1, R2, R3, R4, R5: FANCTL2_R, Resistors_ThroughHole:Resistor_Horizontal_RM10mm, symbol FANCTL2_R
- removed RR?: RR9, symbol RR9
- removed TEMP0: TMP_SNSR_HDR, Pin_Headers:Pin_Header_Straight_2x10, symbol TMP_SNSR_HDR
- added C10, C12: C, Capacitors_ThroughHole:C_Disc_D3_P2.5, symbol C
- added C15: 22n, Capacitors_ThroughHole:C_Disc_D3_P2.5, symbol C
- added D0, D2, D3, D4, D5: D, Diodes_ThroughHole:Diode_DO-35_SOD27_Horizontal_RM10, symbol D
- added JP0, JP1, JP10, JP11, JP2, JP3, JP4, JP5, JP6, JP7, JP8, JP9: JUMPER3, Pin_Headers:Pin_Header_Straight_1x03, symbol JUMPER3
- added P0: CONN_01X03, Pin_Headers:Pin_Header_Straight_1x03, symbol CONN_01X03
- added P2, P3, P4: CONN_01X04, Pin_Headers:Pin_Header_Straight_1x04, symbol CONN_01X04
- added Q7: FAN_NMOS, TO_SOT_Packages_THT:TO-220_Neutral123_Vertical, symbol FAN_NMOS
- added R1: 10K, Resistors_ThroughHole:Resistor_Horizontal_RM10mm, symbol R
- added R15, R16, R17, R18, R19, R20, R21, R22: FANCTL2_R, Resistors_ThroughHole:Resistor_Horizontal_RM10mm, symbol FANCTL2_R
- added R2: 10k, Resistors_ThroughHole:Resistor_Horizontal_RM10mm, symbol R
- added R5: R, Resistors_ThroughHole:Resistor_Horizontal_RM10mm, symbol R
- added RR1: RR8, Housings_SIP:SIP9_Housing, symbol RR8
- added TEMP1: TMP_SNSR_HDR, Pin_Headers:Pin_Header_Straight_2x08, symbol TMP_SNSR_HDR
- added U2: LM358, Housings_DIP:DIP-8_W7.62mm, symbol LM358
- added U3: P82B96, Housings_DIP:DIP-8_W7.62mm, symbol P82B96
- C0, C1, C13, C14, C2, C3, C4, C5, C8, C9: value Decoupler -> 0.1u
- C6, C7: value Decoupler -> 22p
- D1: renamed from D?; footprint (none) -> Diodes_ThroughHole:Diode_DO-35_SOD27_Horizontal_RM10
- L1: value INDUCTOR_SMALL -> 10uH
- Q1, Q2, Q3, Q4, Q5: footprint (none) -> TO_SOT_Packages_THT:TO-220_Neutral123_Vertical
- R3: renamed from R?; footprint (none) -> Resistors_ThroughHole:Resistor_Horizontal_RM10mm
- R4: renamed from R?; value R -> 10k; footprint (none) -> Resistors_ThroughHole:Resistor_Horizontal_RM10mm
- R6: value FANCTL2_R -> 10K
- R7, R8: value FANCTL2_R -> 68
- renumbered D5 to D10, D1 to D11, D0 to D12, D2 to D7, D3 to D8, D4 to D9, JP6 to JP12
Connections:
- net labels added: 12VGND, COM5V, I12V, I5V, SCL, SDA
- wire segments 177 -> 290
- no-connect marks 4 -> 3
Other:
- moved on the sheet: C1, C11, C9, D1, D10, D6, D8, D9, F1, I2C0, L1, P1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
